Commit message: needed some changes for avoidance. needs tuning and a bit of cleaning

File: asv_description/urdf/asv.urdf (robot description, URDF)
Before this commit: robot asv, 1 links, 0 joints
Links:
- link asv: geometry visual mesh filename=package://asv_description/urdf/ferry_shape.STL scale=1 0.1 0.167
