Commit message: First usv implementation. Dynamic model and aitsmc both seem correct from first tests.

File: asv_description/urdf/usv.urdf (robot description, URDF)
Before this commit: robot asv, 1 links, 0 joints
Links:
- removed link asv
- added link usv; visual mesh filename=package://asv_description/models/usv/meshes/asv.dae scale=1 1 1
